Commit message: S

File: urdf/sweepee/sweepee.xacro (robot description, xacro)
@@ -26,5 +26,5 @@
         <origin xyz="0 0 0.032" rpy="0 0 -${M_PI/2}" />
         <geometry>
-          <mesh filename="package://lampo_description/meshes/sweepee/visual/sweepee.dae"/>
+          <mesh filename="file://$(find lampo_description)//meshes/sweepee/visual/sweepee.dae"/>
         </geometry>
         <material name="Gray">
@@ -55,8 +55,6 @@
       <child link="${prefix}rear_laser" />
     </joint>
-  <gazebo reference="${prefix}rear_laser">
+  <!-- <gazebo reference="${prefix}rear_laser">
       <sensor type="ray" name="$(arg prefix)rear_laser">
-          <!-- <pose>0 0 0 0 0 0</pose> -->
-          <!-- <visualize>false</visualize> -->
           <update_rate>10</update_rate>
           <ray>
@@ -75,5 +73,4 @@
           </ray>
           <plugin filename="libgazebo_ros_ray_sensor.so" name="rear_laser_plugin">
-              <!-- <robotNamespace></robotNamespace> -->
               <noise>
                   <type>gaussian</type>
@@ -87,14 +84,11 @@
               <alwaysOn>true</alwaysOn>
               <updateRate>15</updateRate>
-              <!-- <frameName>rear_laser</frameName> -->
               <frame_name>${prefix}rear_laser</frame_name>
               <output_type>sensor_msgs/LaserScan</output_type>
           </plugin>
       </sensor>
-  </gazebo>
-<gazebo reference="${prefix}front_laser">
+  </gazebo> -->
+<!-- <gazebo reference="${prefix}front_laser">
       <sensor type="ray" name="${prefix}front_laser">
-          <!-- <pose>0 0 0 0 0 0</pose> -->
-          <!-- <visualize>false</visualize> -->
           <update_rate>10</update_rate>
           <ray>
@@ -113,5 +107,4 @@
           </ray>
           <plugin filename="libgazebo_ros_ray_sensor.so" name="front_laser_plugin">
-              <!-- <robotNamespace></robotNamespace> -->
               <noise>
                   <type>gaussian</type>
@@ -125,10 +118,38 @@
               <alwaysOn>true</alwaysOn>
               <updateRate>15</updateRate>
-              <!-- <frameName>front_laser</frameName> -->
               <frame_name>${prefix}front_laser</frame_name>
               <output_type>sensor_msgs/LaserScan</output_type>
           </plugin>
       </sensor>
-  </gazebo>
+  </gazebo> -->
+<!-- <gazebo reference="${prefix}front_laser" >
+  <sensor name="${prefix}front_laser" type="gpu_lidar">
+    <topic>scan</topic>
+    <update_rate>30</update_rate>
+    <lidar>
+      <scan>
+        <horizontal>
+          <samples>2800</samples>
+          <resolution>1</resolution>
+          <min_angle>-2.09</min_angle>
+          <max_angle>2.09</max_angle>
+        </horizontal>
+        <vertical>
+          <samples>1</samples>
+          <resolution>0.1</resolution>
+          <min_angle>0.0</min_angle>
+          <max_angle>0.0</max_angle>
+        </vertical>
+      </scan>
+      <range>
+        <min>0.05</min>
+        <max>30.0</max>
+        <resolution>0.01</resolution>
+      </range>
+    </lidar>
+    <alwaysOn>1</alwaysOn>
+    <visualize>true</visualize>
+  </sensor>
+</gazebo> -->
   </xacro:macro>
 </robot>

File: urdf/system.urdf.xacro (robot description, xacro)
@@ -43,4 +43,21 @@
   <!-- convert to property to use substitution in function -->
   <xacro:property name="initial_positions_file" default="$(arg initial_positions_file)"/>
+  <xacro:property name="M_PI" value="3.14159"/>
+  <xacro:sweepee  prefix="$(arg prefix)">
+    <origin xyz="0 0 0" rpy="0 0 0" />
+  </xacro:sweepee>
+  <xacro:sweepee_gazebo />
+  <xacro:if value="$(arg sim_gazebo)">
+    <gazebo reference="world">
+    </gazebo>
+    <gazebo>
+      <plugin filename="libgazebo_ros2_control.so" name="gazebo_ros2_control">
+        <robot_param>robot_description</robot_param>
+        <robot_namespace>$(arg prefix)</robot_namespace>
+        <parameters>$(arg simulation_controllers)</parameters>
+        <robot_param_node>robot_state_publisher</robot_param_node>
+      </plugin>
+    </gazebo>
+  </xacro:if>
    <!-- arm -->
   <xacro:ur_robot
@@ -78,17 +95,5 @@
     <origin xyz="0 0 0" rpy="0 0 0" />
   </xacro:ur_robot>
-  <xacro:if value="$(arg sim_gazebo)">
-    <gazebo reference="world">
-    </gazebo>
-    <gazebo>
-      <plugin filename="libgazebo_ros2_control.so" name="gazebo_ros2_control">
-        <robot_param>robot_description</robot_param>
-        <robot_namespace>$(arg prefix)</robot_namespace>
-        <parameters>$(arg simulation_controllers)</parameters>
-        <robot_param_node>robot_state_publisher</robot_param_node>
-      </plugin>
-    </gazebo>
-  </xacro:if>
-  <!-- <xacro:if value="$(arg sim_ignition)">
+  <xacro:if value="$(arg sim_ignition)">
     <gazebo reference="world">
     </gazebo>
@@ -97,12 +102,10 @@
         <parameters>$(arg simulation_controllers)</parameters>
         <controller_manager_node_name>$(arg prefix)controller_manager</controller_manager_node_name>
+        <robot_param>robot_description</robot_param>
+        <robot_namespace>$(arg prefix)</robot_namespace>
+        <robot_param_node>robot_state_publisher</robot_param_node>
       </plugin>
     </gazebo>
-  </xacro:if> -->
-  <xacro:property name="M_PI" value="3.14159"/>
-  <xacro:sweepee  prefix="$(arg prefix)">
-    <origin xyz="0 0 0" rpy="0 0 0" />
-  </xacro:sweepee>
-  <xacro:sweepee_gazebo />
+  </xacro:if>
   <joint name="$(arg prefix)lifter" type="fixed">
     <parent link="$(arg prefix)base_footprint"/>
@@ -114,7 +117,4 @@
     <plugin name="object_controller" filename="libgazebo_ros_planar_move.so">
         <ros>
-          <!-- Add a namespace -->
-          <!-- <namespace>/</namespace> -->
-          <!-- Remap the default topic -->
           <argument>~cmd_vel:=custom_cmd_vel</argument>
           <argument>~odom:=custom_odom</argument>

Commit message: S: only mobile robots

File: urdf/sweepee/sweepee.xacro (robot description, xacro)
@@ -11,5 +11,5 @@
     <link name="${prefix}base_footprint">
       <inertial>
-          <mass value="1000" />
+          <mass value="10" />
           <inertia ixx="0.001" ixy="0.01" ixz="0.01" iyy="0.001" iyz="0.01" izz="0.001" />
       </inertial>
@@ -33,6 +33,6 @@
       </visual>
       <inertial>
-          <mass value="4000" />
-          <inertia ixx="1.48454" ixy="0.01" ixz="0.01" iyy="3.02861" iyz="0.01" izz="4.10178" />
+          <mass value="40" />
+          <inertia ixx="0.48454" ixy="0.01" ixz="0.01" iyy="0.02861" iyz="0.01" izz="0.10178" />
       </inertial>
     </link>
@@ -88,6 +88,6 @@
           </plugin>
       </sensor>
-  </gazebo> -->
-<!-- <gazebo reference="${prefix}front_laser">
+  </gazebo>  -->
+  <gazebo reference="${prefix}front_laser">
       <sensor type="ray" name="${prefix}front_laser">
           <update_rate>10</update_rate>
@@ -114,5 +114,5 @@
               <ros>
                 <namespace>${prefix}</namespace>
-                <argument>~out:=${prefix}rear_scan</argument>
+                <argument>~out:=${prefix}front_scan</argument>
               </ros>
               <alwaysOn>true</alwaysOn>
@@ -122,5 +122,5 @@
           </plugin>
       </sensor>
-  </gazebo> -->
+  </gazebo>
 <!-- <gazebo reference="${prefix}front_laser" >
   <sensor name="${prefix}front_laser" type="gpu_lidar">

File: urdf/system.urdf.xacro (robot description, xacro)
@@ -50,10 +50,8 @@
   <xacro:if value="$(arg sim_gazebo)">
     <gazebo reference="world">
-    </gazebo>
-    <gazebo>
       <plugin filename="libgazebo_ros2_control.so" name="gazebo_ros2_control">
         <robot_param>robot_description</robot_param>
         <robot_namespace>$(arg prefix)</robot_namespace>
-	<parameters>$(arg simulation_controllers)</parameters>
+	      <parameters>$(arg simulation_controllers)</parameters>
         <robot_param_node>robot_state_publisher</robot_param_node>
       </plugin>
@@ -61,5 +59,5 @@
   </xacro:if>
    <!-- arm -->
-  <xacro:ur_robot
+  <!-- <xacro:ur_robot
     name="$(arg name)"
     prefix="$(arg prefix)"
@@ -94,5 +92,5 @@
     >
     <origin xyz="0 0 0" rpy="0 0 0" />
-  </xacro:ur_robot>
+  </xacro:ur_robot> -->
   <xacro:if value="$(arg sim_ignition)">
     <gazebo reference="world">
@@ -108,10 +106,10 @@
     </gazebo>
   </xacro:if>
-  <joint name="$(arg prefix)lifter" type="fixed">
+  <!-- <joint name="$(arg prefix)lifter" type="fixed">
     <parent link="$(arg prefix)base_footprint"/>
     <child link="$(arg prefix)base_link"/>
     <origin xyz="0 0 0.28" rpy=" 0 0 0"/>
     <axis xyz="0 0 1"/>
-  </joint>
+  </joint> -->
   <gazebo>
     <plugin name="object_controller" filename="libgazebo_ros_planar_move.so">

Commit message: gz

File: urdf/sweepee/sweepee.xacro (robot description, xacro)
@@ -12,5 +12,5 @@
       <inertial>
           <mass value="10" />
-          <inertia ixx="0.001" ixy="0.01" ixz="0.01" iyy="0.001" iyz="0.01" izz="0.001" />
+          <inertia ixx="1.0" ixy="0.0" ixz="0.0" iyy="1.0" iyz="0.0" izz="1.0"/>
       </inertial>
       <collision>
@@ -89,5 +89,5 @@
       </sensor>
   </gazebo>  -->
-  <gazebo reference="${prefix}front_laser">
+  <!-- <gazebo reference="${prefix}front_laser">
       <sensor type="ray" name="${prefix}front_laser">
           <update_rate>10</update_rate>
@@ -122,34 +122,35 @@
           </plugin>
       </sensor>
+  </gazebo> -->
+  <gazebo reference="${prefix}front_laser">
+    <sensor name='gpu_lidar' type='gpu_lidar'>"
+        <pose relative_to='${prefix}front_laser'>0 0 0 0 0 0</pose>
+        <topic>lidar</topic>
+        <update_rate>10</update_rate>
+        <ray>
+            <scan>
+                <horizontal>
+                    <samples>640</samples>
+                    <resolution>1</resolution>
+                    <min_angle>-1.396263</min_angle>
+                    <max_angle>1.396263</max_angle>
+                </horizontal>
+                <vertical>
+                    <samples>1</samples>
+                    <resolution>0.01</resolution>
+                    <min_angle>0</min_angle>
+                    <max_angle>0</max_angle>
+                </vertical>
+            </scan>
+            <range>
+                <min>0.08</min>
+                <max>10.0</max>
+                <resolution>0.01</resolution>
+            </range>
+        </ray>
+        <always_on>1</always_on>
+        <visualize>true</visualize>
+    </sensor>
   </gazebo>
-<!-- <gazebo reference="${prefix}front_laser" >
-  <sensor name="${prefix}front_laser" type="gpu_lidar">
-    <topic>scan</topic>
-    <update_rate>30</update_rate>
-    <lidar>
-      <scan>
-        <horizontal>
-          <samples>2800</samples>
-          <resolution>1</resolution>
-          <min_angle>-2.09</min_angle>
-          <max_angle>2.09</max_angle>
-        </horizontal>
-        <vertical>
-          <samples>1</samples>
-          <resolution>0.1</resolution>
-          <min_angle>0.0</min_angle>
-          <max_angle>0.0</max_angle>
-        </vertical>
-      </scan>
-      <range>
-        <min>0.05</min>
-        <max>30.0</max>
-        <resolution>0.01</resolution>
-      </range>
-    </lidar>
-    <alwaysOn>1</alwaysOn>
-    <visualize>true</visualize>
-  </sensor>
-</gazebo> -->
   </xacro:macro>
 </robot>

File: urdf/system.urdf.xacro (robot description, xacro)
@@ -34,8 +34,8 @@
   <xacro:arg name="tool_tcp_port" default="54321" />
     <!-- Simulation parameters -->
-  <xacro:arg name="use_fake_hardware" default="false" />
-  <xacro:arg name="fake_sensor_commands" default="false" />
+  <xacro:arg name="use_fake_hardware" default="true" />
+  <xacro:arg name="fake_sensor_commands" default="true" />
   <xacro:arg name="sim_gazebo" default="false" />
-  <xacro:arg name="sim_ignition" default="false" />
+  <xacro:arg name="sim_ignition" default="true" />
   <xacro:arg name="simulation_controllers" default="error_default" />
   <!-- initial position for simulations (Fake Hardware, Gazebo, Ignition) -->
@@ -57,4 +57,11 @@
       </plugin>
     </gazebo>
+  </xacro:if>
+  <xacro:if value="$(arg sim_ignition)">
+    <plugin
+      filename="gz-sim-sensors-system"
+      name="gz::sim::systems::Sensors">
+      <render_engine>ogre2</render_engine>
+    </plugin>
   </xacro:if>
    <!-- arm -->
@@ -91,11 +98,11 @@
     input_recipe_filename="$(arg input_recipe_filename)"
     >
-    <origin xyz="0 0 0" rpy="0 0 0" />
+    <origin xyz="0 0 0.4" rpy="0 0 0" />
   </xacro:ur_robot> -->
   <xacro:if value="$(arg sim_ignition)">
-    <gazebo reference="world">
+    <!-- <gazebo reference="world">
     </gazebo>
-    <gazebo>
-      <plugin filename="libign_ros2_control-system.so" name="ign_ros2_control::IgnitionROS2ControlPlugin">
+    <gazebo> -->
+      <plugin filename="gz_ros2_control-system" name="gz_ros2_control::GazeboSimROS2ControlPlugin">
         <parameters>$(arg simulation_controllers)</parameters>
         <controller_manager_node_name>$(arg prefix)controller_manager</controller_manager_node_name>
@@ -112,5 +119,5 @@
     <axis xyz="0 0 1"/>
   </joint> -->
-  <gazebo>
+  <!-- <gazebo>
     <plugin name="object_controller" filename="libgazebo_ros_planar_move.so">
         <ros>
@@ -128,4 +135,4 @@
         <covariance_yaw>0.01</covariance_yaw>
       </plugin>
-  </gazebo>
+  </gazebo> -->
 </robot>
