Commit message: sdf

File: urdf/sweepee/sweepee.xacro (robot description, xacro)
@@ -1,4 +1,4 @@
 <?xml version="1.0"?>
-<robot name="eureca" xmlns:xacro="http://ros.org/wiki/xacro">
+<robot name="eureca" xmlns:xacro="http://www.ros.org/wiki/xacro" xmlns:gz="http://gazebosim.org/schema">
   <!-- <xacro:include filename="$(find lampo_description)/urdf/sweepee/camera.urdf.xacro" /> -->
   <xacro:property name="M_PI" value="3.14159"/>
@@ -10,14 +10,4 @@
     <!-- Base footprint is on the ground under the robot -->
     <link name="${prefix}base_footprint">
-      <inertial>
-          <mass value="10" />
-          <inertia ixx="1.0" ixy="0.0" ixz="0.0" iyy="1.0" iyz="0.0" izz="1.0"/>
-      </inertial>
-      <collision>
-        <origin xyz="0 0 0.005" rpy="0 0 0" />
-        <geometry>
-          <box size="${base_x_size} ${base_y_size} 0.01"/>
-        </geometry>
-      </collision>
     </link>
     <!-- Base link is the center of the robot's bottom plate -->
@@ -33,7 +23,14 @@
       </visual>
       <inertial>
-          <mass value="40" />
-          <inertia ixx="0.48454" ixy="0.01" ixz="0.01" iyy="0.02861" iyz="0.01" izz="0.10178" />
+          <origin xyz="0 0 0.2" rpy="0 0 0" />
+          <mass value="150" />
+          <inertia ixx="2.0" ixy="0.0" ixz="0.0" iyy="3.7" iyz="0.0" izz="6.0" />
       </inertial>
+      <collision>
+        <origin xyz="0 0 0.2" rpy="0 0 0" />
+        <geometry>
+          <box size="0.3 ${base_y_size} 0.05"/>
+        </geometry>
+      </collision>
     </link>
     <joint name="${prefix}base_footprint_joint" type="fixed">
@@ -41,5 +38,4 @@
       <parent link="${prefix}base_footprint" />
       <child link="${prefix}base_link_sweepee" />
-      <dynamics damping="0.7"/>
     </joint>
     <link name="${prefix}front_laser" />
@@ -55,76 +51,120 @@
       <child link="${prefix}rear_laser" />
     </joint>
-  <!-- <gazebo reference="${prefix}rear_laser">
-      <sensor type="ray" name="$(arg prefix)rear_laser">
-          <update_rate>10</update_rate>
-          <ray>
-              <scan display="false">
-                  <horizontal>
-                      <samples>750</samples>
-                      <resolution>1</resolution>
-                      <min_angle>-${M_PI /2}</min_angle>
-                      <max_angle> ${M_PI /2}</max_angle>
-                  </horizontal>
-              </scan>
-              <range>
-                  <min>0.25</min>
-                  <max>59.0</max>
-              </range>
-          </ray>
-          <plugin filename="libgazebo_ros_ray_sensor.so" name="rear_laser_plugin">
-              <noise>
-                  <type>gaussian</type>
-                  <mean>0.0</mean>
-                  <stddev>0.01</stddev>
-              </noise>
-              <ros>
-                <namespace>${prefix}</namespace>
-                <argument>~out:=${prefix}rear_scan</argument>
-              </ros>
-              <alwaysOn>true</alwaysOn>
-              <updateRate>15</updateRate>
-              <frame_name>${prefix}rear_laser</frame_name>
-              <output_type>sensor_msgs/LaserScan</output_type>
-          </plugin>
-      </sensor>
-  </gazebo>  -->
-  <!-- <gazebo reference="${prefix}front_laser">
-      <sensor type="ray" name="${prefix}front_laser">
-          <update_rate>10</update_rate>
-          <ray>
-              <scan display="false">
-                  <horizontal>
-                      <samples>750</samples>
-                      <resolution>1</resolution>
-                      <min_angle>-${M_PI /2}</min_angle>
-                      <max_angle> ${M_PI /2}</max_angle>
-                  </horizontal>
-              </scan>
-              <range>
-                  <min>0.25</min>
-                  <max>59.0</max>
-              </range>
-          </ray>
-          <plugin filename="libgazebo_ros_ray_sensor.so" name="front_laser_plugin">
-              <noise>
-                  <type>gaussian</type>
-                  <mean>0.0</mean>
-                  <stddev>0.01</stddev>
-              </noise>
-              <ros>
-                <namespace>${prefix}</namespace>
-                <argument>~out:=${prefix}front_scan</argument>
-              </ros>
-              <alwaysOn>true</alwaysOn>
-              <updateRate>15</updateRate>
-              <frame_name>${prefix}front_laser</frame_name>
-              <output_type>sensor_msgs/LaserScan</output_type>
-          </plugin>
-      </sensor>
-  </gazebo> -->
+      <link name='${prefix}front_left_wheel'>
+        <inertial>
+          <mass value="1"/>
+          <inertia ixx="0.145"  ixy="0"  ixz="0" iyy="0.145" iyz="0" izz="0.125" />
+        </inertial>
+        <visual>
+          <geometry>
+            <sphere length="0.05" radius="0.1"/>
+          </geometry>
+        </visual>
+        <collision>
+          <geometry>
+            <sphere length="0.05" radius="0.1"/>
+          </geometry>
+        </collision>
+      </link>
+      <link name='${prefix}rear_left_wheel'>
+        <inertial>
+          <mass value="1"/>
+          <inertia ixx="0.145"  ixy="0"  ixz="0" iyy="0.145" iyz="0" izz="0.125" />
+        </inertial>
+        <visual>
+          <geometry>
+            <sphere length="0.05" radius="0.1"/>
+          </geometry>
+        </visual>
+        <collision>
+          <geometry>
+            <sphere length="0.05" radius="0.1"/>
+          </geometry>
+        </collision>
+      </link>
+      <link name='${prefix}front_right_wheel'>
+        <inertial>
+          <mass value="1"/>
+          <inertia ixx="0.145"  ixy="0"  ixz="0" iyy="0.145" iyz="0" izz="0.125" />
+        </inertial>
+        <visual>
+          <geometry>
+            <sphere length="0.05" radius="0.1"/>
+          </geometry>
+        </visual>
+        <collision>
+          <geometry>
+            <sphere length="0.05" radius="0.1"/>
+          </geometry>
+        </collision>
+      </link>
+      <link name='${prefix}rear_right_wheel'>
+        <inertial>
+          <mass value="1"/>
+          <inertia ixx="0.145"  ixy="0"  ixz="0" iyy="0.145" iyz="0" izz="0.125" />
+        </inertial>
+        <visual>
+          <geometry>
+            <sphere length="0.05" radius="0.1"/>
+          </geometry>
+        </visual>
+        <collision>
+          <geometry>
+            <sphere length="0.05" radius="0.1"/>
+          </geometry>
+        </collision>
+      </link>
+      <gazebo reference="${prefix}front_left_wheel">
+        <mu1>1.0</mu1>
+        <mu2>0.0</mu2>
+        <fdir1 gz:expressed_in='${prefix}base_footprint'>1 -1 0</fdir1>
+      </gazebo>
+      <gazebo reference="${prefix}rear_left_wheel">
+        <mu1>1.0</mu1>
+        <mu2>0.0</mu2>
+        <fdir1 gz:expressed_in='${prefix}base_footprint'>1 1 0</fdir1>
+      </gazebo>
+      <gazebo reference="${prefix}front_right_wheel">
+        <mu1>1.0</mu1>
+        <mu2>0.0</mu2>
+        <fdir1 gz:expressed_in='${prefix}base_footprint'>1 1 0</fdir1>
+      </gazebo>
+        <gazebo reference="${prefix}rear_right_wheel">
+        <mu1>1.0</mu1>
+        <mu2>0.0</mu2>
+        <fdir1 gz:expressed_in='${prefix}base_footprint'>1 -1 0</fdir1>
+      </gazebo>
+      <joint name='${prefix}front_left_wheel_joint' type='revolute'>
+        <origin xyz="0.3 0.25 0.1" rpy="-1.5707 0 0"/>
+        <parent link="${prefix}base_link_sweepee"/>
+        <child link="${prefix}front_left_wheel"/>
+        <axis xyz="0 0 1"/>
+        <limit effort="10000.0" lower="-1.79769e+308" upper="1.79769e+308" velocity="5.1"/>
+      </joint>
+      <joint name='${prefix}front_right_wheel_joint' type='revolute'>
+        <origin xyz="0.3 -0.25 0.1" rpy="-1.5707 0 0"/>
+        <parent link="${prefix}base_link_sweepee"/>
+        <child link="${prefix}front_right_wheel"/>
+        <axis xyz="0 0 1"/>
+        <limit effort="10000.0" lower="-1.79769e+308" upper="1.79769e+308" velocity="5.1"/>
+      </joint>
+      <joint name='${prefix}rear_left_wheel_joint' type='revolute'>
+        <origin xyz="-0.3 0.25 0.1" rpy="-1.5707 0 0"/>
+        <parent link="${prefix}base_link_sweepee"/>
+        <child link="${prefix}rear_left_wheel"/>
+        <axis xyz="0 0 1"/>
+        <limit effort="10000.0" lower="-1.79769e+308" upper="1.79769e+308" velocity="5.1"/>
+      </joint>
+      <joint name='${prefix}rear_right_wheel_joint' type='revolute'>
+        <origin xyz="-0.3 -0.25 0.1" rpy="-1.5707 0 0"/>
+        <parent link="${prefix}base_link_sweepee"/>
+        <child link="${prefix}rear_right_wheel"/>
+        <axis xyz="0 0 1"/>
+        <limit effort="10000.0" lower="-1.79769e+308" upper="1.79769e+308" velocity="5.1"/>
+      </joint>
   <gazebo reference="${prefix}front_laser">
     <sensor name='gpu_lidar' type='gpu_lidar'>"
         <pose relative_to='${prefix}front_laser'>0 0 0 0 0 0</pose>
-        <topic>lidar</topic>
+        <topic>${prefix}lidar</topic>
         <update_rate>10</update_rate>
         <ray>
@@ -153,4 +193,21 @@
     </sensor>
   </gazebo>
+  <gazebo>
+    <plugin
+      filename="gz-sim-mecanum-drive-system"
+      name="gz::sim::systems::MecanumDrive">
+      <front_left_joint>${prefix}front_left_wheel_joint</front_left_joint>
+      <front_right_joint>${prefix}front_right_wheel_joint</front_right_joint>
+      <back_left_joint>${prefix}rear_left_wheel_joint</back_left_joint>
+      <back_right_joint>${prefix}rear_right_wheel_joint</back_right_joint>
+      <wheel_separation>0.5</wheel_separation>
+      <wheelbase>0.7</wheelbase>
+      <wheel_radius>0.1</wheel_radius>
+      <min_acceleration>-5</min_acceleration>
+      <max_acceleration>5</max_acceleration>
+      <topic>${prefix}cmd_vel</topic>
+      <frame_id>${prefix}base_link_sweepee</frame_id>
+    </plugin>
+  </gazebo>
   </xacro:macro>
 </robot>

File: urdf/system.urdf.xacro (robot description, xacro)
@@ -1,4 +1,4 @@
 <?xml version="1.0"?>
-<robot name="eureca" xmlns:xacro="http://ros.org/wiki/xacro">
+<robot name="mobile_manipulator" xmlns:xacro="http://ros.org/wiki/xacro" xmlns:gz="http://gazebosim.org/schema">>
   <xacro:include filename="$(find lampo_description)/urdf/sweepee/sweepee.gazebo.xacro" />
   <xacro:include filename="$(find lampo_description)/urdf/sweepee/sweepee.xacro" />
@@ -112,13 +112,4 @@
         </plugin>
     </gazebo>
-    <!-- <gazebo>
-      <plugin filename="gz_ros2_control-system" name="gz_ros2_control::GazeboSimROS2ControlPlugin">
-        <parameters>$(arg simulation_controllers)</parameters>
-        <controller_manager_node_name>$(arg prefix)controller_manager</controller_manager_node_name>
-        <robot_param>robot_description</robot_param>
-        <robot_namespace>$(arg prefix)</robot_namespace>
-        <robot_param_node>robot_state_publisher</robot_param_node>
-      </plugin>
-    </gazebo> -->
   </xacro:if>
   <!-- <joint name="$(arg prefix)lifter" type="fixed">

Commit message: Harmonic fix

File: urdf/sweepee/sweepee.xacro (robot description, xacro)
@@ -10,9 +10,9 @@
     <!-- Base footprint is on the ground under the robot -->
     <link name="${prefix}base_footprint">
-        <inertial>
+        <!-- <inertial>
           <origin xyz="0 0 0.0" rpy="0 0 0" />
           <mass value="150" />
           <inertia ixx="2.0" ixy="0.01" ixz="0.01" iyy="3.7" iyz="0.01" izz="6.0" />
-      </inertial>
+      </inertial> -->
     </link>
     <!-- Base link is the center of the robot's bottom plate -->
@@ -44,14 +44,26 @@
       <child link="${prefix}base_link_sweepee" />
     </joint>
-    <link name="${prefix}front_laser" />
-    <joint name="${prefix}front_laser_joint" type="fixed">
+    <link name="${prefix}front_laser">
+      <inertial>
+        <mass value="5"/>
+        <inertia ixx="0.145"  ixy="0"  ixz="0" iyy="0.145" iyz="0" izz="0.125" />
+      </inertial>
+      <visual>
+        <geometry>
+          <sphere length="0.005" radius="0.1"/>
+        </geometry>
+      </visual>
+    </link>
+    <joint name="${prefix}front_laser_joint" type="revolute">
       <origin xyz="${base_x_size/2-0.15} 0.0 ${base_z_size/2+0.085}" rpy="0 0 0" />
-      <parent link="${prefix}base_link_sweepee" />
+      <parent link="${prefix}base_footprint" />
       <child link="${prefix}front_laser" />
+      <axis xyz="0 0 1"/>
+      <limit effort="10000.0" lower="-1.79769e+308" upper="1.79769e+308" velocity="5.1"/>
     </joint>
       <link name="${prefix}rear_laser" />
     <joint name="${prefix}rear_laser_joint" type="fixed">
       <origin xyz="${-base_x_size/2+0.15} 0.0 ${base_z_size/2+0.085}" rpy="0 0 ${M_PI}" />
-      <parent link="${prefix}base_link_sweepee" />
+      <parent link="${prefix}base_footprint" />
       <child link="${prefix}rear_laser" />
     </joint>
@@ -169,11 +181,9 @@
       </joint>
   <gazebo reference="${prefix}front_laser">
-  <!-- <gazebo> -->
     <sensor name='gpu_lidar' type='gpu_lidar'>"
-        <!-- <pose relative_to='${prefix}front_laser'>0 0 0 0 0 0</pose> -->
-        <pose relative_to='asd'>0 0 0 0 0 0</pose>
+        <pose relative_to='${prefix}front_laser'>0 0 0 0 0 0</pose>
+        <gz_frame_id>${prefix}front_laser</gz_frame_id>
         <topic>${prefix}lidar</topic>
         <update_rate>10</update_rate>
-        <frame_id>asdasd</frame_id>
         <ray>
             <scan>
@@ -199,4 +209,9 @@
         <always_on>1</always_on>
         <visualize>true</visualize>
+        <!-- <plugin
+            filename="gz-sim-sensors-system"
+            name="gz::sim::systems::Sensors">
+        <render_engine>ogre2</render_engine>
+        </plugin> -->
     </sensor>
   </gazebo>

Commit message: fixed sim time , still lidar error

File: urdf/sweepee/sweepee.xacro (robot description, xacro)
@@ -55,10 +55,8 @@
       </visual>
     </link>
-    <joint name="${prefix}front_laser_joint" type="revolute">
+    <joint name="${prefix}front_laser_joint" type="fixed">
       <origin xyz="${base_x_size/2-0.15} 0.0 ${base_z_size/2+0.085}" rpy="0 0 0" />
       <parent link="${prefix}base_footprint" />
-      <child link="${prefix}front_laser" />
-      <axis xyz="0 0 1"/>
-      <limit effort="10000.0" lower="-1.79769e+308" upper="1.79769e+308" velocity="5.1"/>
+      <child link="${prefix}front_laser" /> -->
     </joint>
       <link name="${prefix}rear_laser" />
