Commit message: diff almost ok, lack tf

File: urdf/sweepee/sweepee_diff.xacro (robot description, xacro)
@@ -1,5 +1,4 @@
 <?xml version="1.0"?>
 <robot name="eureca" xmlns:xacro="http://www.ros.org/wiki/xacro" xmlns:gz="http://gazebosim.org/schema">
-  <!-- <xacro:include filename="$(find lampo_description)/urdf/sweepee/camera.urdf.xacro" /> -->
   <xacro:property name="M_PI" value="3.14159"/>
   <!-- Base Size -->
@@ -10,9 +9,4 @@
     <!-- Base footprint is on the ground under the robot -->
     <link name="${prefix}base_footprint">
-        <!-- <inertial>
-          <origin xyz="0 0 0.0" rpy="0 0 0" />
-          <mass value="150" />
-          <inertia ixx="2.0" ixy="0.01" ixz="0.01" iyy="3.7" iyz="0.01" izz="6.0" />
-      </inertial> -->
     </link>
     <!-- Base link is the center of the robot's bottom plate -->
@@ -57,5 +51,5 @@
     <joint name="${prefix}front_laser_joint" type="fixed">
       <origin xyz="${base_x_size/2-0.15} 0.0 ${base_z_size/2+0.085}" rpy="0 0 0" />
-      <parent link="${prefix}base_footprint" />
+      <parent link="${prefix}base_link_sweepee" />
       <child link="${prefix}front_laser" /> -->
     </joint>
@@ -63,5 +57,5 @@
     <joint name="${prefix}rear_laser_joint" type="fixed">
       <origin xyz="${-base_x_size/2+0.15} 0.0 ${base_z_size/2+0.085}" rpy="0 0 ${M_PI}" />
-      <parent link="${prefix}base_footprint" />
+      <parent link="${prefix}base_link_sweepee" />
       <child link="${prefix}rear_laser" />
     </joint>
@@ -130,7 +124,7 @@
         </collision>
       </link>
-      <gazebo reference="${prefix}front_left_wheel">
-        <mu1>5.0</mu1>
-        <mu2>1.0</mu2>
+      <!-- <gazebo reference="${prefix}front_left_wheel">
+        <mu1>0.5</mu1>
+        <mu2>0.1</mu2>
         <fdir1 gz:expressed_in='${prefix}base_footprint'>1 -1 0</fdir1>
       </gazebo>
@@ -141,12 +135,62 @@
       </gazebo>
       <gazebo reference="${prefix}front_right_wheel">
-        <mu1>5.0</mu1>
-        <mu2>1.0</mu2>
+        <mu1>0.5</mu1>
+        <mu2>0.1</mu2>
         <fdir1 gz:expressed_in='${prefix}base_footprint'>1 1 0</fdir1>
       </gazebo>
-        <gazebo reference="${prefix}rear_right_wheel">
+      <gazebo reference="${prefix}rear_right_wheel">
         <mu1>0.0</mu1>
         <mu2>0.0</mu2>
         <fdir1 gz:expressed_in='${prefix}base_footprint'>1 -1 0</fdir1>
+      </gazebo> -->
+      <gazebo reference='${prefix}front_left_wheel'>
+        <collision>
+          <surface>
+            <friction>
+              <ode>
+                <mu>0.7</mu>
+                <mu2>0.3</mu2>
+                <!-- <fdir1 gz:expressed_in="sweepee_1/base_footprint">1 0 0</fdir1> -->
+              </ode>
+            </friction>
+          </surface>
+        </collision>
+      </gazebo>
+      <gazebo reference='${prefix}front_right_wheel'>
+        <collision>
+          <surface>
+            <friction>
+              <ode>
+                <mu>0.7</mu>
+                <mu2>0.3</mu2>
+                <!-- <fdir1 gz:expressed_in="sweepee_1/base_footprint">1 0 0</fdir1> -->
+              </ode>
+            </friction>
+          </surface>
+        </collision>
+      </gazebo>
+      <gazebo reference='${prefix}rear_left_wheel'>
+        <collision>
+          <surface>
+            <friction>
+              <ode>
+                <mu>0.0</mu>
+                <mu2>0.0</mu2>
+              </ode>
+            </friction>
+          </surface>
+        </collision>
+      </gazebo>
+      <gazebo reference='${prefix}rear_right_wheel'>
+        <collision>
+          <surface>
+            <friction>
+              <ode>
+                <mu>0.0</mu>
+                <mu2>0.0</mu2>
+              </ode>
+            </friction>
+          </surface>
+        </collision>
       </gazebo>
       <joint name='${prefix}front_left_wheel_joint' type='revolute'>
@@ -209,22 +253,4 @@
     </sensor>
   </gazebo>
-  <!-- <gazebo>
-    <plugin
-      filename="gz-sim-mecanum-drive-system"
-      name="gz::sim::systems::MecanumDrive">
-      <front_left_joint>${prefix}front_left_wheel_joint</front_left_joint>
-      <front_right_joint>${prefix}front_right_wheel_joint</front_right_joint>
-      <back_left_joint>${prefix}rear_left_wheel_joint</back_left_joint>
-      <back_right_joint>${prefix}rear_right_wheel_joint</back_right_joint>
-      <wheel_separation>0.5</wheel_separation>
-      <wheelbase>0.7</wheelbase>
-      <wheel_radius>0.1</wheel_radius>
-      <min_acceleration>-5</min_acceleration>
-      <max_acceleration>5</max_acceleration>
-      <topic>${prefix}cmd_vel</topic>
-      <frame_id>${prefix}base_footprint</frame_id>
-      <odom_topic>${prefix}odom</odom_topic>
-    </plugin>
-  </gazebo> -->
   <gazebo>
       <plugin

File: urdf/system.urdf.xacro (robot description, xacro)
@@ -1,6 +1,11 @@
 <?xml version="1.0"?>
 <robot name="mm1" xmlns:xacro="http://ros.org/wiki/xacro" xmlns:gz="http://gazebosim.org/schema">>
-  <xacro:include filename="$(find lampo_description)/urdf/sweepee/sweepee.gazebo.xacro" />
-  <xacro:include filename="$(find lampo_description)/urdf/sweepee/sweepee.xacro" />
+  <xacro:arg name="omni" default="false" />
+  <xacro:if value="$(arg omni)">
+    <xacro:include filename="$(find lampo_description)/urdf/sweepee/sweepee_omni.xacro" />
+  </xacro:if>
+  <xacro:unless value="$(arg omni)">
+    <xacro:include filename="$(find lampo_description)/urdf/sweepee/sweepee_diff.xacro" />
+  </xacro:unless>
   <xacro:arg name="name" default="ur"/>
   <xacro:include filename="$(find ur_description)/urdf/ur_macro.xacro"/>
@@ -46,5 +51,5 @@
     <origin xyz="0 0 0" rpy="0 0 0" />
   </xacro:sweepee>
-  <xacro:sweepee_gazebo />
+  <!-- <xacro:sweepee_gazebo /> -->
    <!-- arm -->
   <xacro:if value="$(arg mm)">

Commit message: fixed drift and TF

File: urdf/sweepee/sweepee_diff.xacro (robot description, xacro)
@@ -23,6 +23,6 @@
       <inertial>
           <origin xyz="0 0 0.2" rpy="0 0 0" />
-          <mass value="150" />
-          <inertia ixx="2.0" ixy="0.0" ixz="0.0" iyy="3.7" iyz="0.0" izz="6.0" />
+          <mass value="250" />
+          <inertia ixx="12.0" ixy="0.0" ixz="0.0" iyy="12.0" iyz="0.0" izz="12.0" />
       </inertial>
       <collision>
@@ -45,5 +45,5 @@
       <visual>
         <geometry>
-          <sphere length="0.005" radius="0.1"/>
+          <cylinder length="0.005" radius="0.1"/>
         </geometry>
       </visual>
@@ -67,10 +67,10 @@
         <visual>
           <geometry>
-            <sphere length="0.05" radius="0.1"/>
-          </geometry>
-        </visual>
-        <collision>
-          <geometry>
-            <sphere length="0.05" radius="0.1"/>
+            <cylinder length="0.05" radius="0.1"/>
+          </geometry>
+        </visual>
+        <collision>
+          <geometry>
+            <cylinder length="0.05" radius="0.1"/>
           </geometry>
         </collision>
@@ -83,10 +83,10 @@
         <visual>
           <geometry>
-            <sphere length="0.05" radius="0.1"/>
-          </geometry>
-        </visual>
-        <collision>
-          <geometry>
-            <sphere length="0.05" radius="0.1"/>
+            <cylinder length="0.05" radius="0.1"/>
+          </geometry>
+        </visual>
+        <collision>
+          <geometry>
+            <cylinder length="0.05" radius="0.1"/>
           </geometry>
         </collision>
@@ -99,10 +99,10 @@
         <visual>
           <geometry>
-            <sphere length="0.05" radius="0.1"/>
-          </geometry>
-        </visual>
-        <collision>
-          <geometry>
-            <sphere length="0.05" radius="0.1"/>
+            <cylinder length="0.05" radius="0.1"/>
+          </geometry>
+        </visual>
+        <collision>
+          <geometry>
+            <cylinder length="0.05" radius="0.1"/>
           </geometry>
         </collision>
@@ -115,10 +115,10 @@
         <visual>
           <geometry>
-            <sphere length="0.05" radius="0.1"/>
-          </geometry>
-        </visual>
-        <collision>
-          <geometry>
-            <sphere length="0.05" radius="0.1"/>
+            <cylinder length="0.05" radius="0.1"/>
+          </geometry>
+        </visual>
+        <collision>
+          <geometry>
+            <cylinder length="0.05" radius="0.1"/>
           </geometry>
         </collision>
@@ -175,6 +175,6 @@
             <friction>
               <ode>
-                <mu>0.0</mu>
-                <mu2>0.0</mu2>
+                <mu>0.05</mu>
+                <mu2>0.01</mu2>
               </ode>
             </friction>
@@ -187,6 +187,6 @@
             <friction>
               <ode>
-                <mu>0.0</mu>
-                <mu2>0.0</mu2>
+                <mu>0.05</mu>
+                <mu2>0.01</mu2>
               </ode>
             </friction>

Commit message: fixings on omni

File: urdf/sweepee/sweepee_diff.xacro (robot description, xacro)
@@ -151,5 +151,4 @@
                 <mu>0.7</mu>
                 <mu2>0.3</mu2>
-                <!-- <fdir1 gz:expressed_in="sweepee_1/base_footprint">1 0 0</fdir1> -->
               </ode>
             </friction>
@@ -164,5 +163,4 @@
                 <mu>0.7</mu>
                 <mu2>0.3</mu2>
-                <!-- <fdir1 gz:expressed_in="sweepee_1/base_footprint">1 0 0</fdir1> -->
               </ode>
             </friction>
@@ -199,5 +197,5 @@
         <child link="${prefix}front_left_wheel"/>
         <axis xyz="0 0 1"/>
-        <limit effort="10000.0" lower="-1.79769e+308" upper="1.79769e+308" velocity="5.1"/>
+        <limit effort="10000.0" lower="-1.79769e+308" upper="1.79769e+308" velocity="15.1"/>
       </joint>
       <joint name='${prefix}front_right_wheel_joint' type='revolute'>
@@ -206,5 +204,5 @@
         <child link="${prefix}front_right_wheel"/>
         <axis xyz="0 0 1"/>
-        <limit effort="10000.0" lower="-1.79769e+308" upper="1.79769e+308" velocity="5.1"/>
+        <limit effort="10000.0" lower="-1.79769e+308" upper="1.79769e+308" velocity="15.1"/>
       </joint>
       <joint name='${prefix}rear_left_wheel_joint' type='revolute'>
@@ -213,5 +211,5 @@
         <child link="${prefix}rear_left_wheel"/>
         <axis xyz="0 0 1"/>
-        <limit effort="10000.0" lower="-1.79769e+308" upper="1.79769e+308" velocity="5.1"/>
+        <limit effort="10000.0" lower="-1.79769e+308" upper="1.79769e+308" velocity="15.1"/>
       </joint>
       <joint name='${prefix}rear_right_wheel_joint' type='revolute'>
@@ -220,5 +218,5 @@
         <child link="${prefix}rear_right_wheel"/>
         <axis xyz="0 0 1"/>
-        <limit effort="10000.0" lower="-1.79769e+308" upper="1.79769e+308" velocity="5.1"/>
+        <limit effort="10000.0" lower="-1.79769e+308" upper="1.79769e+308" velocity="15.1"/>
       </joint>
   <gazebo reference="${prefix}front_laser">

File: urdf/sweepee/sweepee_omni.xacro (robot description, xacro)
@@ -1,5 +1,4 @@
 <?xml version="1.0"?>
 <robot name="eureca" xmlns:xacro="http://www.ros.org/wiki/xacro" xmlns:gz="http://gazebosim.org/schema">
-  <!-- <xacro:include filename="$(find lampo_description)/urdf/sweepee/camera.urdf.xacro" /> -->
   <xacro:property name="M_PI" value="3.14159"/>
   <!-- Base Size -->
@@ -10,9 +9,4 @@
     <!-- Base footprint is on the ground under the robot -->
     <link name="${prefix}base_footprint">
-        <!-- <inertial>
-          <origin xyz="0 0 0.0" rpy="0 0 0" />
-          <mass value="150" />
-          <inertia ixx="2.0" ixy="0.01" ixz="0.01" iyy="3.7" iyz="0.01" izz="6.0" />
-      </inertial> -->
     </link>
     <!-- Base link is the center of the robot's bottom plate -->
@@ -29,6 +23,6 @@
       <inertial>
           <origin xyz="0 0 0.2" rpy="0 0 0" />
-          <mass value="150" />
-          <inertia ixx="2.0" ixy="0.0" ixz="0.0" iyy="3.7" iyz="0.0" izz="6.0" />
+          <mass value="250" />
+          <inertia ixx="12.0" ixy="0.0" ixz="0.0" iyy="12.0" iyz="0.0" izz="12.0" />
       </inertial>
       <collision>
@@ -51,5 +45,5 @@
       <visual>
         <geometry>
-          <sphere length="0.005" radius="0.1"/>
+          <cylinder length="0.005" radius="0.1"/>
         </geometry>
       </visual>
@@ -73,10 +67,10 @@
         <visual>
           <geometry>
-            <sphere length="0.05" radius="0.1"/>
-          </geometry>
-        </visual>
-        <collision>
-          <geometry>
-            <sphere length="0.05" radius="0.1"/>
+            <cylinder length="0.05" radius="0.1"/>
+          </geometry>
+        </visual>
+        <collision>
+          <geometry>
+            <cylinder length="0.05" radius="0.1"/>
           </geometry>
         </collision>
@@ -89,10 +83,10 @@
         <visual>
           <geometry>
-            <sphere length="0.05" radius="0.1"/>
-          </geometry>
-        </visual>
-        <collision>
-          <geometry>
-            <sphere length="0.05" radius="0.1"/>
+            <cylinder length="0.05" radius="0.1"/>
+          </geometry>
+        </visual>
+        <collision>
+          <geometry>
+            <cylinder length="0.05" radius="0.1"/>
           </geometry>
         </collision>
@@ -105,10 +99,10 @@
         <visual>
           <geometry>
-            <sphere length="0.05" radius="0.1"/>
-          </geometry>
-        </visual>
-        <collision>
-          <geometry>
-            <sphere length="0.05" radius="0.1"/>
+            <cylinder length="0.05" radius="0.1"/>
+          </geometry>
+        </visual>
+        <collision>
+          <geometry>
+            <cylinder length="0.05" radius="0.1"/>
           </geometry>
         </collision>
@@ -121,10 +115,10 @@
         <visual>
           <geometry>
-            <sphere length="0.05" radius="0.1"/>
-          </geometry>
-        </visual>
-        <collision>
-          <geometry>
-            <sphere length="0.05" radius="0.1"/>
+            <cylinder length="0.05" radius="0.1"/>
+          </geometry>
+        </visual>
+        <collision>
+          <geometry>
+            <cylinder length="0.05" radius="0.1"/>
           </geometry>
         </collision>
@@ -155,7 +149,7 @@
             <friction>
               <ode>
-                <mu>0.7</mu>
-                <mu2>0.3</mu2>
-                <fdir1 gz:expressed_in="sweepee_1/base_footprint">1 -1 0</fdir1>
+                <mu>1.0</mu>
+                <mu2>0.0</mu2>
+                <fdir1 gz:expressed_in="${prefix}base_footprint">1 -1 0</fdir1>
               </ode>
             </friction>
@@ -168,7 +162,7 @@
             <friction>
               <ode>
-                <mu>0.7</mu>
-                <mu2>0.3</mu2>
-                <fdir1 gz:expressed_in="sweepee_1/base_footprint">1 1 0</fdir1>
+                <mu>1.0</mu>
+                <mu2>0.0</mu2>
+                <fdir1 gz:expressed_in="${prefix}base_footprint">1 1 0</fdir1>
               </ode>
             </friction>
@@ -181,7 +175,7 @@
             <friction>
               <ode>
-                <mu>0.0</mu>
-                <mu2>0.0</mu2>
-                <fdir1 gz:expressed_in="sweepee_1/base_footprint">1 1 0</fdir1>
+                <mu>1.0</mu>
+                <mu2>0.0</mu2>
+                <fdir1 gz:expressed_in="${prefix}base_footprint">1 1 0</fdir1>
               </ode>
             </friction>
@@ -194,7 +188,7 @@
             <friction>
               <ode>
-                <mu>0.0</mu>
-                <mu2>0.0</mu2>
-                <fdir1 gz:expressed_in="sweepee_1/base_footprint">1 -1 0</fdir1>
+                <mu>1.0</mu>
+                <mu2>0.0</mu2>
+                <fdir1 gz:expressed_in="${prefix}base_footprint">1 -1 0</fdir1>
               </ode>
             </friction>
@@ -207,5 +201,5 @@
         <child link="${prefix}front_left_wheel"/>
         <axis xyz="0 0 1"/>
-        <limit effort="10000.0" lower="-1.79769e+308" upper="1.79769e+308" velocity="5.1"/>
+        <limit effort="10000.0" lower="-1.79769e+308" upper="1.79769e+308" velocity="15.1"/>
       </joint>
       <joint name='${prefix}front_right_wheel_joint' type='revolute'>
@@ -214,5 +208,5 @@
         <child link="${prefix}front_right_wheel"/>
         <axis xyz="0 0 1"/>
-        <limit effort="10000.0" lower="-1.79769e+308" upper="1.79769e+308" velocity="5.1"/>
+        <limit effort="10000.0" lower="-1.79769e+308" upper="1.79769e+308" velocity="15.1"/>
       </joint>
       <joint name='${prefix}rear_left_wheel_joint' type='revolute'>
@@ -221,5 +215,5 @@
         <child link="${prefix}rear_left_wheel"/>
         <axis xyz="0 0 1"/>
-        <limit effort="10000.0" lower="-1.79769e+308" upper="1.79769e+308" velocity="5.1"/>
+        <limit effort="10000.0" lower="-1.79769e+308" upper="1.79769e+308" velocity="15.1"/>
       </joint>
       <joint name='${prefix}rear_right_wheel_joint' type='revolute'>
@@ -228,5 +222,5 @@
         <child link="${prefix}rear_right_wheel"/>
         <axis xyz="0 0 1"/>
-        <limit effort="10000.0" lower="-1.79769e+308" upper="1.79769e+308" velocity="5.1"/>
+        <limit effort="10000.0" lower="-1.79769e+308" upper="1.79769e+308" velocity="15.1"/>
       </joint>
   <gazebo reference="${prefix}front_laser">
@@ -252,6 +246,6 @@
             </scan>
             <range>
-                <min>0.08</min>
-                <max>10.0</max>
+                <min>0.15</min>
+                <max>30.0</max>
                 <resolution>0.01</resolution>
             </range>
@@ -270,11 +264,14 @@
       <back_right_joint>${prefix}rear_right_wheel_joint</back_right_joint>
       <wheel_separation>0.5</wheel_separation>
-      <wheelbase>0.7</wheelbase>
+      <wheelbase>0.6</wheelbase>
       <wheel_radius>0.1</wheel_radius>
       <min_acceleration>-5</min_acceleration>
       <max_acceleration>5</max_acceleration>
+      <max_velocity>1.5</max_velocity>
       <topic>${prefix}cmd_vel</topic>
-      <frame_id>${prefix}base_footprint</frame_id>
+      <frame_id>${prefix}odom</frame_id>
       <odom_topic>${prefix}odom</odom_topic>
+      <child_frame_id>${prefix}base_footprint</child_frame_id>
+      <tf_topic>tf</tf_topic>
     </plugin>
   </gazebo>
